Commit message: Testing which geometries create contact points
THe first test confirms that only a two conditions will produce contact
points.  Very small spheres and boxes (with special testing for evaluating
the definition of "small".)

File: drake/multibody/test/rigid_body_tree/contact_points_generation.urdf (robot description, URDF)
Before this commit: robot contact_point_generator, 1 links, 0 joints
Links:
- link body: geometry collision box size=2 2 2; collision capsule length=1 radius=0.5
