Commit message: Correct anchored test
Floating bodies only remain floating if they: a) have inertia or b) have
children.

I added inertia so those tests pass.

File: drake/multibody/test/rigid_body_tree/anchored_parentless_link.urdf (robot description, URDF)
Before this commit: robot simple_anchored, 1 links, 0 joints
Links:
- link parentless_body: mass None -> 1
