Commit message: Using polytop urdf (and converted sdf). Passive dynamics matches. Problem with controller

File: manipulation/models/iiwa_description/urdf/iiwa14_no_collision.urdf (robot description, URDF)
Before this commit: robot iiwa14, 11 links, 10 joints
Links:
- removed link base
Joints:
- removed joint iiwa_base_joint
- joint iiwa_joint_1: limit lower=-2.96705972839 upper=2.96705972839 effort=300 velocity=10 -> effort=300 velocity=10
- joint iiwa_joint_2: limit lower=-2.09439510239 upper=2.09439510239 effort=300 velocity=10 -> effort=300 velocity=10
- joint iiwa_joint_3: limit lower=-2.96705972839 upper=2.96705972839 effort=300 velocity=10 -> effort=300 velocity=10
- joint iiwa_joint_4: limit lower=-2.09439510239 upper=2.09439510239 effort=300 velocity=10 -> effort=300 velocity=10
- joint iiwa_joint_5: limit lower=-2.96705972839 upper=2.96705972839 effort=300 velocity=10 -> effort=300 velocity=10
- joint iiwa_joint_6: limit lower=-2.09439510239 upper=2.09439510239 effort=300 velocity=10 -> effort=300 velocity=10
- joint iiwa_joint_7: limit lower=-3.05432619099 upper=3.05432619099 effort=300 velocity=10 -> effort=300 velocity=10
